File: pcb/address_bus_buff.kicad_sch (KiCad schematic)
At the start: 25 parts, among them U23 74AHCT541, U24 74AHCT541, U25 74AHCT541

Commit message: comment
Connections:
- net A21: now also U25.5 (A3)
- net A22: now also U25.6 (A4)
- net A23: now also U25.7 (A5)
- net SA21: now also U25.15 (Y3)
- net SA22: now also U25.14 (Y4)
- net SA23: now also U25.13 (Y5)
- no-connect marks 16 -> 10
Other:
- note added: "74HC573 better?"
Changed lines of the file:
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@@
 		(members "SA[2..23]")
 	)
-	(no_connect
-		(at 205.74 96.52)
+	(text "74HC573 better?"
+		(exclude_from_sim no)
+		(at 155.194 55.626 0)
+		(effects
+			(font
+				(size 5 5)
+			)
+		)
 	)
 	(no_connect
@@
 	)
 	(no_connect
-		(at 205.74 93.98)
-	)
-	(no_connect
-		(at 231.14 91.44)
-	)
-	(no_connect
-		(at 205.74 91.44)
-	)
-	(no_connect
 		(at 231.14 99.06)
 	)
@@
 	)
 	(no_connect
-		(at 231.14 93.98)
-	)
-	(no_connect
 		(at 205.74 99.06)
 	)
@@
 		(at 104.14 106.68)
 	)
-	(no_connect
-		(at 231.14 96.52)
+	(bus_entry
+		(at 200.66 93.98)
+		(size -2.54 -2.54)
+		(stroke
+			(width 0)
+			(type default)
+		)
 	)
 	(bus_entry
@@
 	)
 	(bus_entry
+		(at 200.66 91.44)
+		(size -2.54 -2.54)
+		(stroke
+			(width 0)
+			(type default)
+		)
+	)
+	(bus_entry
+		(at 236.22 91.44)
+		(size 2.54 -2.54)
+		(stroke
+			(width 0)
+			(type default)
+		)
+	)
+	(bus_entry
+		(at 200.66 96.52)
+		(size -2.54 -2.54)
+		(stroke
+			(width 0)
+			(type default)
+		)
+	)
+	(bus_entry
 		(at 60.96 73.66)
 		(size -2.54 -2.54)
@@
 	)
 	(bus_entry
+		(at 236.22 93.98)
+		(size 2.54 -2.54)
+		(stroke
+			(width 0)
+			(type default)
+		)
+	)
+	(bus_entry
 		(at 236.22 83.82)
 		(size 2.54 -2.54)
@@
 	)
 	(bus_entry
+		(at 236.22 96.52)
+		(size 2.54 -2.54)
+		(stroke
+			(width 0)
+			(type default)
+		)
+	)
+	(bus_entry
 		(at 83.82 73.66)
 		(size 2.54 -2.54)
@@
 	(wire
 		(pts
+			(xy 200.66 96.52) (xy 205.74 96.52)
+		)
+		(stroke
+			(width 0)
+			(type default)
+		)
+	)
+	(wire
+		(pts
 			(xy 74.93 73.66) (xy 83.82 73.66)
 		)
@@
 	(bus
 		(pts
+			(xy 198.12 91.44) (xy 198.12 88.9)
+		)
+		(stroke
+			(width 0)
+			(type default)
+		)
+	)
+	(bus
+		(pts
 			(xy 58.42 78.74) (xy 58.42 76.2)
 		)
@@
 	(bus
 		(pts
+			(xy 238.76 88.9) (xy 238.76 86.36)
+		)
+		(stroke
+			(width 0)
+			(type default)
+		)
+	)
+	(bus
+		(pts
 			(xy 58.42 45.72) (xy 58.42 55.88)
 		)
@@
 		)
 	)
+	(wire
+		(pts
+			(xy 231.14 96.52) (xy 236.22 96.52)
+		)
+		(stroke
+			(width 0)
+			(type default)
+		)
+	)
 	(bus
 		(pts
@@
 		)
 	)
+	(wire
+		(pts
+			(xy 200.66 91.44) (xy 205.74 91.44)
+		)
+		(stroke
+			(width 0)
+			(type default)
+		)
+	)
 	(bus
 		(pts
@@
 		)
 	)
+	(wire
+		(pts
+			(xy 231.14 91.44) (xy 236.22 91.44)
+		)
+		(stroke
+			(width 0)
+			(type default)
+		)
+	)
 	(bus
 		(pts
@@
 		)
 	)
+	(bus
+		(pts
+			(xy 238.76 91.44) (xy 238.76 88.9)
+		)
+		(stroke
+			(width 0)
+			(type default)
+		)
+	)
+	(bus
+		(pts
+			(xy 198.12 88.9) (xy 198.12 86.36)
+		)
+		(stroke
+			(width 0)
+			(type default)
+		)
+	)
 	(wire
 		(pts
@@
 	(wire
 		(pts
+			(xy 200.66 93.98) (xy 205.74 93.98)
+		)
+		(stroke
+			(width 0)
+			(type default)
+		)
+	)
+	(wire
+		(pts
 			(xy 74.93 83.82) (xy 83.82 83.82)
 		)
@@
 		)
 	)
+	(bus
+		(pts
+			(xy 198.12 93.98) (xy 198.12 91.44)
+		)
+		(stroke
+			(width 0)
+			(type default)
+		)
+	)
 	(wire
 		(pts
@@
 	(wire
 		(pts
+			(xy 231.14 93.98) (xy 236.22 93.98)
+		)
+		(stroke
+			(width 0)
+			(type default)
+		)
+	)
+	(wire
+		(pts
 			(xy 60.96 81.28) (xy 69.85 81.28)
 		)
@@
 		)
 	)
+	(bus
+		(pts
+			(xy 238.76 93.98) (xy 238.76 91.44)
+		)
+		(stroke
+			(width 0)
+			(type default)
+		)
+	)
+	(label "A22"
+		(at 200.66 93.98 0)
+		(effects
+			(font
+				(size 1.27 1.27)
+			)
+			(justify left bottom)
+		)
+	)
 	(label "A13"
 		(at 149.86 91.44 0)
@@
 		)
 	)
+	(label "A21"
+		(at 200.66 91.44 0)
+		(effects
+			(font
+				(size 1.27 1.27)
+			)
+			(justify left bottom)
+		)
+	)
 	(label "A2"
 		(at 60.96 58.42 0)
@@
 		)
 	)
+	(label "SA23"
+		(at 236.22 96.52 180)
+		(effects
+			(font
+				(size 1.27 1.27)
+			)
+			(justify right bottom)
+		)
+	)
 	(label "A20"
 		(at 60.96 104.14 0)
@@
 		)
 	)
+	(label "SA21"
+		(at 236.22 91.44 180)
+		(effects
+			(font
+				(size 1.27 1.27)
+			)
+			(justify right bottom)
+		)
+	)
 	(label "A4"
 		(at 60.96 63.5 0)
@@
 		)
 	)
+	(label "A23"
+		(at 200.66 96.52 0)
+		(effects
+			(font
+				(size 1.27 1.27)
+			)
+			(justify left bottom)
+		)
+	)
 	(label "A11"
 		(at 60.96 81.28 0)
@@
 		)
 	)
+	(label "SA22"
+		(at 236.22 93.98 180)
+		(effects
+			(font
+				(size 1.27 1.27)
+			)
+			(justify right bottom)
+		)
+	)
